File: PCB/spin.sch (EAGLE design)
At the start: 19 parts

Commit message: edited spin pcb resistor value for android communication
Parts:
- R5: value 100 -> 1k
Connections:
- net N$4 renamed RED
- net N$5 renamed GREEN
- net N$6 renamed YELLOW
- net N$7 renamed BLUE
Changed lines of the file:
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@@
 <part name="GND3" library="SparkFun-Aesthetics" deviceset="GND" device=""/>
 <part name="R4" library="rcl" deviceset="R-US_" device="R1206" value="1k"/>
-<part name="R5" library="rcl" deviceset="R-US_" device="R1206" value="100"/>
+<part name="R5" library="rcl" deviceset="R-US_" device="R1206" value="1k"/>
 <part name="SUPPLY1" library="SparkFun-Aesthetics" deviceset="VCC" device=""/>
 <part name="GND4" library="SparkFun-Aesthetics" deviceset="GND" device=""/>
@@
 </segment>
 </net>
-<net name="N$4" class="0">
+<net name="RED" class="0">
 <segment>
 <pinref part="EASY_DRIVER" gate="G$1" pin="B1"/>
@@
 <wire x1="86.36" y1="38.1" x2="91.44" y2="38.1" width="0.1524" layer="91"/>
 <junction x="86.36" y="38.1"/>
-</segment>
-</net>
-<net name="N$5" class="0">
+<label x="86.36" y="38.1" size="1.778" layer="95"/>
+</segment>
+</net>
+<net name="GREEN" class="0">
 <segment>
 <pinref part="EASY_DRIVER" gate="G$1" pin="B2"/>
@@
 <wire x1="86.36" y1="35.56" x2="91.44" y2="35.56" width="0.1524" layer="91"/>
 <junction x="86.36" y="35.56"/>
-</segment>
-</net>
-<net name="N$6" class="0">
+<label x="86.36" y="35.56" size="1.778" layer="95"/>
+</segment>
+</net>
+<net name="YELLOW" class="0">
 <segment>
 <pinref part="EASY_DRIVER" gate="G$1" pin="A2"/>
@@
 <wire x1="86.36" y1="33.02" x2="91.44" y2="33.02" width="0.1524" layer="91"/>
 <junction x="86.36" y="33.02"/>
-</segment>
-</net>
-<net name="N$7" class="0">
+<label x="86.36" y="33.02" size="1.778" layer="95"/>
+</segment>
+</net>
+<net name="BLUE" class="0">
 <segment>
 <pinref part="EASY_DRIVER" gate="G$1" pin="A1"/>
@@
 <wire x1="86.36" y1="30.48" x2="91.44" y2="30.48" width="0.1524" layer="91"/>
 <junction x="86.36" y="30.48"/>
-</segment>
-</net>
+<label x="86.36" y="30.48" size="1.778" layer="95"/>
+</segment>
+</net>
